File: PCB_Design/ee463_project/ee463_project.kicad_sch (KiCad schematic)
At the start: 16 parts, among them Q1 C2M0080120D, U1 TLP250, U2 L7808

Commit message: PCB Completed Gerber Files Added
Parts:
- added C8: 1n, Capacitor_SMD:C_0603_1608Metric, symbol Device:C_Small
- added C9: 100n, Capacitor_SMD:C_0603_1608Metric, symbol Device:C_Small
- added D3: LED, Resistor_SMD:R_0603_1608Metric, symbol Device:LED
- added R4, R5, R6, R7: 0, Resistor_SMD:R_1206_3216Metric, symbol Device:R
- added R8: 1k, Resistor_SMD:R_0603_1608Metric, symbol Device:R
- added U3: ACS712xLCTR-30A, Package_SO:SOIC-8_3.9x4.9mm_P1.27mm, symbol Sensor_Current:ACS712xLCTR-30A
- C1, C2, C3, C6, C7: footprint Capacitor_SMD:C_0504_1310Metric -> Capacitor_SMD:C_1206_3216Metric
Connections:
- net GND is gone; now on net GND1: U1.3 (C)
- net GND1: now also C8.2, C9.2, D3.1 (K), U3.5 (GND)
- net V_in_arduino: now also R5.2; no longer C7.1, U2.3 (OUT)
- net Vcc: now also R4.1; no longer C6.1, U2.1 (IN)
- net at A1.19 (A0): now also R7.1
- net at A1.27 (+5V): now also R6.1
- new net: C9.1, R6.2, R8.1, U3.8 (VCC)
- new net: C7.1, R5.1, U2.3 (OUT)
- new net: C6.1, R4.2, U2.1 (IN)
- new net: D3.2 (A), R8.2
- new net: R7.2, U3.7 (VIOUT)
- new net: C8.1, U3.6 (FILTER)
- new net OUT+: U3.1 (IP+), U3.2 (IP+)
- new net OUT-: U3.3 (IP-), U3.4 (IP-)

Commit message: PCB Design Updated
Parts:
- added H1, H2, H3, H4: MountingHole, MountingHole:MountingHole_2.2mm_M2, symbol Mechanical:MountingHole
Changed lines of the file:
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@@
     (pin "3")
+  )
+  (symbol (lib_id "Mechanical:MountingHole") (at 96.52 153.67 0) (unit 1)
+    (in_bom yes) (on_board yes) (fields_autoplaced)
+    (property "Reference" "H3" (id 0) (at 99.06 152.3999 0)
+      (effects (font (size 1.27 1.27)) (justify left))
+    )
+    (property "Value" "MountingHole" (id 1) (at 99.06 154.9399 0)
+      (effects (font (size 1.27 1.27)) (justify left))
+    )
+    (property "Footprint" "MountingHole:MountingHole_2.2mm_M2" (id 2) (at 96.52 153.67 0)
+      (effects (font (size 1.27 1.27)) hide)
+    )
+    (property "Datasheet" "~" (id 3) (at 96.52 153.67 0)
+      (effects (font (size 1.27 1.27)) hide)
+    )
   )
   (symbol (lib_id "Device:C_Small") (at 73.66 64.77 0) (unit 1)
@@
     (pin "2")
   )
+  (symbol (lib_id "Mechanical:MountingHole") (at 73.66 153.67 0) (unit 1)
+    (in_bom yes) (on_board yes) (fields_autoplaced)
+    (property "Reference" "H2" (id 0) (at 76.2 152.3999 0)
+      (effects (font (size 1.27 1.27)) (justify left))
+    )
+    (property "Value" "MountingHole" (id 1) (at 76.2 154.9399 0)
+      (effects (font (size 1.27 1.27)) (justify left))
+    )
+    (property "Footprint" "MountingHole:MountingHole_2.2mm_M2" (id 2) (at 73.66 153.67 0)
+      (effects (font (size 1.27 1.27)) hide)
+    )
+    (property "Datasheet" "~" (id 3) (at 73.66 153.67 0)
+      (effects (font (size 1.27 1.27)) hide)
+    )
+  )
   (symbol (lib_id "Device:R") (at 83.82 102.87 90) (unit 1)
     (in_bom yes) (on_board yes) (fields_autoplaced)
@@
     (pin "2")
   )
+  (symbol (lib_id "Mechanical:MountingHole") (at 50.8 153.67 0) (unit 1)
+    (in_bom yes) (on_board yes) (fields_autoplaced)
+    (property "Reference" "H1" (id 0) (at 53.34 152.3999 0)
+      (effects (font (size 1.27 1.27)) (justify left))
+    )
+    (property "Value" "MountingHole" (id 1) (at 53.34 154.9399 0)
+      (effects (font (size 1.27 1.27)) (justify left))
+    )
+    (property "Footprint" "MountingHole:MountingHole_2.2mm_M2" (id 2) (at 50.8 153.67 0)
+      (effects (font (size 1.27 1.27)) hide)
+    )
+    (property "Datasheet" "~" (id 3) (at 50.8 153.67 0)
+      (effects (font (size 1.27 1.27)) hide)
+    )
+  )
   (symbol (lib_id "Device:C_Small") (at 252.73 92.71 0) (unit 1)
     (in_bom yes) (on_board yes) (fields_autoplaced)
@@
     (pin "1")
     (pin "2")
+  )
+  (symbol (lib_id "Mechanical:MountingHole") (at 120.65 153.67 0) (unit 1)
+    (in_bom yes) (on_board yes) (fields_autoplaced)
+    (property "Reference" "H4" (id 0) (at 123.19 152.3999 0)
+      (effects (font (size 1.27 1.27)) (justify left))
+    )
+    (property "Value" "MountingHole" (id 1) (at 123.19 154.9399 0)
+      (effects (font (size 1.27 1.27)) (justify left))
+    )
+    (property "Footprint" "MountingHole:MountingHole_2.2mm_M2" (id 2) (at 120.65 153.67 0)
+      (effects (font (size 1.27 1.27)) hide)
+    )
+    (property "Datasheet" "~" (id 3) (at 120.65 153.67 0)
+      (effects (font (size 1.27 1.27)) hide)
+    )
   )
   (symbol (lib_id "Device:R") (at 92.71 107.95 0) (unit 1)
@@
       (reference "D3") (unit 1) (value "LED") (footprint "Resistor_SMD:R_0603_1608Metric")
     )
+    (path "/afdaf757-4872-48e6-b235-66a2236e5bb7"
+      (reference "H1") (unit 1) (value "MountingHole") (footprint "MountingHole:MountingHole_2.2mm_M2")
+    )
+    (path "/87df9e64-d645-488e-b2da-eb492d54e2df"
+      (reference "H2") (unit 1) (value "MountingHole") (footprint "MountingHole:MountingHole_2.2mm_M2")
+    )
+    (path "/510a3876-3213-4b70-863f-068df27b7abf"
+      (reference "H3") (unit 1) (value "MountingHole") (footprint "MountingHole:MountingHole_2.2mm_M2")
+    )
+    (path "/c41dfda2-f31a-4c46-93b8-0114b30b25ef"
+      (reference "H4") (unit 1) (value "MountingHole") (footprint "MountingHole:MountingHole_2.2mm_M2")
+    )
     (path "/e27aa64a-eb67-416d-95d0-9472e552ada2"
