File: PCB_Design/ee463_project/ee463_project.kicad_pcb (KiCad board)
At the start: 2 copper layers, 180.3 x 123.2 mm, 16 parts, among them Q1 C2M0080120D, U1 TLP250, U2 L7808

Commit message: PCB Completed Gerber Files Added
Parts:
- added C8: 1n, Capacitor_SMD:C_0603_1608Metric, F.Cu at (118.6, 117.1)
- added C9: 100n, Capacitor_SMD:C_0603_1608Metric, F.Cu at (106.4, 129.9)
- added D3: LED, Resistor_SMD:R_0603_1608Metric, F.Cu at (104.9, 133.0)
- added R4: 0, Resistor_SMD:R_1206_3216Metric, F.Cu at (166.4, 101.9)
- added R5: 0, Resistor_SMD:R_1206_3216Metric, F.Cu at (152.4, 108.2)
- added R6: 0, Resistor_SMD:R_1206_3216Metric, F.Cu at (104.9, 125.7)
- added R7: 0, Resistor_SMD:R_1206_3216Metric, F.Cu at (113.5, 116.8)
- added R8: 1k, Resistor_SMD:R_0603_1608Metric, F.Cu at (104.1, 130.0)
- added U3: ACS712xLCTR-30A, Package_SO:SOIC-8_3.9x4.9mm_P1.27mm, F.Cu at (117.3, 125.2)
- C1, C2, C3, C6, C7: footprint Capacitor_SMD:C_0504_1310Metric -> Capacitor_SMD:C_1206_3216Metric
- moved A1 29.1 mm to (141.5, 94.5), turned to -90 degrees
- moved C6 6.62 mm to (164.8, 97.5)
- moved C7 6.62 mm to (152.4, 100.3)
- moved U2 6.06 mm to (164.8, 106.5)
- moved C2 4.67 mm to (169.7, 89.7), turned to 180 degrees
- moved C3 4.60 mm to (169.4, 96.3)
- moved C1 4.35 mm to (169.7, 93.0)
- moved R3 4.06 mm to (175.5, 84.3)
- moved D1 1.91 mm to (153.3, 54.2), turned to -30 degrees
Connections:
- A1 pad 19: unconnected-(A1-Pad19) -> Net-(A1-Pad19)
- A1 pad 27: unconnected-(A1-Pad27) -> Net-(A1-Pad27)
- C6 pad 1: Vcc -> Net-(C6-Pad1)
- C7 pad 1: V_in_arduino -> Net-(C7-Pad1)
- U1 pad 3: GND -> GND1
- U2 pad 1: Vcc -> Net-(C6-Pad1)
- U2 pad 3: V_in_arduino -> Net-(C7-Pad1)
Routing:
- net PWM: track 0.00 -> 175.1 mm
- net Net-(A1-Pad27): track 0.00 -> 50.9 mm
- net Net-(U3-Pad8): track 0.00 -> 17.2 mm
- net Net-(C7-Pad1): track 0.00 -> 12.4 mm
- net V_in_arduino: track 0.00 -> 11.0 mm
- net Net-(R2-Pad1): track 0.00 -> 8.72 mm
- net Net-(C6-Pad1): track 0.00 -> 7.54 mm
- net Net-(U3-Pad7): track 0.00 -> 6.91 mm
- net Net-(U3-Pad6): track 0.00 -> 5.71 mm
- net Net-(A1-Pad19): track 0.00 -> 5.64 mm
- net Net-(R1-Pad2): track 0.00 -> 2.36 mm
- net Net-(D3-Pad2): track 0.00 -> 2.19 mm
- added copper zone on F.Cu, net GND1
- added copper zone on F.Cu, net Gate
- added copper zone on F.Cu, net OUT+
- added copper zone on F.Cu, net OUT-
- added copper zone on F.Cu, net Vcc
Other:
- board size 180.3 x 123.2 mm -> 159.3 x 123.2 mm

Commit message: PCB Design Updated
Parts:
- added H1: MountingHole, MountingHole:MountingHole_2.2mm_M2, F.Cu at (54.4, 133.4)
- added H2: MountingHole, MountingHole:MountingHole_2.2mm_M2, F.Cu at (161.3, 27.4)
- added H3: MountingHole, MountingHole:MountingHole_2.2mm_M2, F.Cu at (54.4, 27.4)
- added H4: MountingHole, MountingHole:MountingHole_2.2mm_M2, F.Cu at (162.6, 133.6)
- moved R1 39.9 mm to (137.2, 112.5), turned to 0 degrees
- moved U1 32.1 mm to (142.5, 105.4), turned to 0 degrees
- moved C3 31.2 mm to (138.2, 96.3)
- moved Q1 31.2 mm to (145.8, 74.4)
- moved R3 31.2 mm to (144.3, 84.3)
- moved R4 31.2 mm to (135.1, 101.9)
- moved C1 31.2 mm to (138.4, 93.0)
- moved C2 31.2 mm to (138.4, 89.7)
- moved C4 31.2 mm to (109.2, 55.4)
- moved C5 31.2 mm to (94.7, 55.7)
- moved C6 31.2 mm to (133.6, 97.5)
- moved D1 31.2 mm to (122.0, 54.2)
- moved R2 31.2 mm to (145.7, 92.5)
- moved U2 31.2 mm to (133.6, 106.5)
- moved R5 29.3 mm to (123.2, 106.4), turned to 180 degrees
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Routing:
- net Net-(R2-Pad1): track 8.72 -> 35.5 mm
- net PWM: track 175.1 -> 156.1 mm
- net Net-(R1-Pad2): track 2.36 -> 7.67 mm
- net V_in_arduino: track 11.0 -> 7.13 mm
- net Net-(C7-Pad1): track 12.4 -> 11.1 mm
Other:
- board size 159.3 x 123.2 mm -> 124 x 121.9 mm

Commit message: PCB Design Updated
Parts:
- removed C8: 1n, Capacitor_SMD:C_0603_1608Metric
- removed C9: 100n, Capacitor_SMD:C_0603_1608Metric
- removed D3: LED, Resistor_SMD:R_0603_1608Metric
- removed R4, R5, R6, R7: 0, Resistor_SMD:R_1206_3216Metric
- removed R8: 1k, Resistor_SMD:R_0603_1608Metric
- removed U3: ACS712xLCTR-30A, Package_SO:SOIC-8_3.9x4.9mm_P1.27mm
- A1, D1, D2, Q1, U2: moved to B.Cu
- C4, C5: footprint Capacitor_THT:C_Radial_D10.0mm_H16.0mm_P5.00mm -> Capacitor_THT:CP_Radial_D35.0mm_P10.00mm_SnapIn; moved to B.Cu
- H1, H2, H3, H4: footprint MountingHole:MountingHole_2.2mm_M2 -> MountingHole:MountingHole_4.3mm_M4
- moved A1 38.1 mm to (108.7, 128.3), turned to 90 degrees
- moved D1 30.5 mm to (152.6, 54.5), turned to -135 degrees
- moved C5 27.5 mm to (122.2, 54.6)
- moved C4 24.7 mm to (84.6, 53.7)
- moved R1 20.3 mm to (132.6, 132.3)
- moved U1 17.9 mm to (140.0, 123.2), turned to 90 degrees
- moved Q1 14.4 mm to (156.6, 83.9)
- moved C7 13.6 mm to (117.7, 106.1)
- moved R3 13.6 mm to (154.9, 92.7)
- moved R2 13.0 mm to (157.2, 98.6)
- moved D2 8.13 mm to (59.7, 51.0), turned to 180 degrees
- moved U2 8.01 mm to (127.5, 111.7)
- moved C6 7.89 mm to (131.6, 105.2)
- moved C3 6.62 mm to (138.7, 102.9)
- moved C1 6.36 mm to (138.8, 99.3)
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Connections:
- A1 pad 12: PWM -> unconnected-(A1-Pad12)
- A1 pad 19: Net-(A1-Pad19) -> OUT
- A1 pad 27: Net-(A1-Pad27) -> +5V
- A1 pad 8: unconnected-(A1-Pad8) -> PWM
- C6 pad 1: Net-(C6-Pad1) -> Vcc
- C7 pad 1: Net-(C7-Pad1) -> V_in_arduino
- U2 pad 1: Net-(C6-Pad1) -> Vcc
- U2 pad 3: Net-(C7-Pad1) -> V_in_arduino
Routing:
- net PWM: track 156.1 -> 43.7 mm
- net +5V: track 0.00 -> 60.1 mm
- net Net-(A1-Pad27): track 50.9 -> 0.00 mm
- net OUT: track 0.00 -> 43.7 mm
- net Net-(C9-Pad1): track 17.2 -> 0.00 mm
- net Net-(C7-Pad1): track 11.1 -> 0.00 mm
- net Net-(C6-Pad1): track 7.54 -> 0.00 mm
- net V_in_arduino: track 7.13 -> 0.00 mm
- net Net-(R7-Pad2): track 6.91 -> 0.00 mm
- net Net-(R1-Pad2): track 7.67 -> 14.6 mm
- net Net-(C8-Pad1): track 5.71 -> 0.00 mm
- net Net-(A1-Pad19): track 5.64 -> 0.00 mm
- net Net-(D3-Pad2): track 2.19 -> 0.00 mm
- net Net-(R2-Pad1): track 35.5 -> 37.2 mm
- added copper zone on F.Cu, net V_in_arduino
- removed copper zone on F.Cu, net OUT+
- removed copper zone on F.Cu, net OUT-
