File: PCB_Design/ee463_project/v1.0/ee463_project.kicad_sch (KiCad schematic)
At the start: 20 parts, among them Q1 C2M0080120D, U1 TLP250, U2 L7808

Commit message: PCB Design Updated
Parts:
- added C8: 1n, Capacitor_SMD:C_0603_1608Metric, symbol Device:C_Small
- added C9: 100n, Capacitor_SMD:C_0603_1608Metric, symbol Device:C_Small
- added D3: LED, Resistor_SMD:R_0603_1608Metric, symbol Device:LED
- added R4, R5, R6, R7: 0, Resistor_SMD:R_1206_3216Metric, symbol Device:R
- added R8: 1k, Resistor_SMD:R_0603_1608Metric, symbol Device:R
- added U3: ACS712xLCTR-30A, Package_SO:SOIC-8_3.9x4.9mm_P1.27mm, symbol Sensor_Current:ACS712xLCTR-30A
- C4, C5: footprint Capacitor_THT:CP_Radial_D35.0mm_P10.00mm_SnapIn -> Capacitor_THT:C_Radial_D10.0mm_H16.0mm_P5.00mm
- H1, H2, H3, H4: footprint MountingHole:MountingHole_4.3mm_M4 -> MountingHole:MountingHole_2.2mm_M2
Connections:
- net GND1: now also C8.2, C9.2, D3.1 (K), U3.5 (GND)
- net PWM: now also A1.12 (D9); no longer A1.8 (D5)
- net V_in_arduino: now also R5.2; no longer C7.1, U2.3 (OUT)
- net Vcc: now also R4.1; no longer C6.1, U2.1 (IN)
- net +5V: no longer names the net of A1.27 (+5V)
- net +5V: now also R6.1
- net OUT: no longer names the net of A1.19 (A0)
- net OUT: now also R7.1
- new net: C9.1, R6.2, R8.1, U3.8 (VCC)
- new net: C7.1, R5.1, U2.3 (OUT)
- new net: C6.1, R4.2, U2.1 (IN)
- new net: D3.2 (A), R8.2
- new net: R7.2, U3.7 (VIOUT)
- new net: C8.1, U3.6 (FILTER)
- new net OUT+: U3.1 (IP+), U3.2 (IP+)
- new net OUT-: U3.3 (IP-), U3.4 (IP-)
